File: schematics/picotouch_synth_flip.brd (EAGLE design)
At the start: 253.8 x 41.6 mm, 100 parts, among them IC1 H11L1MS, J1 AUDIO-JACK-TRRS, J2 AUDIO-JACK-TRRS, J3 AUDIO-JACK-TRRS, U1 RASPBERRY_PICOSMD

Commit message: flip version updates
Parts:
- moved J3 1.27 mm to (0.00, 31.8)
- moved J2 1.27 mm to (0.00, 11.4)
- moved C21 0.51 mm to (21.6, 18.5)
- moved R23 0.51 mm to (18.8, 18.5)
- moved R24 0.51 mm to (16.0, 18.5)
Routing:
- net GP28: track 33.0 -> 39.9 mm
- net GP27: track 47.5 -> 41.1 mm
- net GND: track 40.1 -> 36.7 mm
- net PWM_AUDIO: track 237.6 -> 235.1 mm
- net AUDIO_OUT: track 18.8 -> 17.7 mm
- net N$6: track 16.0 -> 15.3 mm
- net N$4: track 12.6 -> 11.9 mm
- net N$3: track 20.8 -> 20.3 mm
- net MIDI_IN: track 217.4 -> 216.9 mm
- net MIDI_OUT: track 220.2 -> 220.7 mm
Other:
- outline, holes or cut-outs redrawn

Commit message: flip version updates
Routing:
- net GP28: track 39.9 -> 35.9 mm
- net +3V3: track 496.9 -> 495.2 mm
- net N$3: track 20.3 -> 21.3 mm
- net N$6: track 15.3 -> 16.2 mm, vias 0 -> 2
- net GP17: track 25.6 -> 24.7 mm
- net MIDI_IN: track 216.9 -> 216.1 mm
- net GP27: track 41.1 -> 40.3 mm
- net GP18: track 33.8 -> 33.2 mm
- net N$4: track 11.9 -> 12.5 mm, vias 0 -> 2
Other:
- board text added: "line out"
- board text added: "midi in"
- board text added: "midi out"
- board text added: "trs-a"
- board text removed: "audio line out"
- board text removed: "midi in (trs-a)"
- board text removed: "midi out (trs-a)"
